Commit message: Pruebas para levantarse y de rozamientos para arreglar caminata

File: pruebas/moving_nao/nao_movement_pattern_creator/Modelo_NAO/nao.urdf (robot description, URDF)
Before this commit: robot NaoH25V50, 79 links, 78 joints
Links:
- link l_ankle: mass 0.17184 -> 1.16184
- link r_ankle: mass 0.17184 -> 1.16184
Joints:
- joint LHipPitch: limit lower=-1.53589 upper=0.48398 effort=3.023 velocity=6.40239 -> lower=-1.53589 upper=1.53589 effort=3.023 velocity=6.40239
- joint LShoulderPitch: limit lower=-2.08567 upper=2.08567 effort=1.329 velocity=8.26797 -> lower=-5.08567 upper=5.08567 effort=1.329 velocity=8.26797
- joint RHipPitch: limit lower=-1.53589 upper=0.48398 effort=3.0226 velocity=6.40239 -> lower=-1.53589 upper=1.53589 effort=3.0226 velocity=6.40239
- joint RShoulderPitch: limit lower=-2.08567 upper=2.08567 effort=1.329 velocity=8.26797 -> lower=-5.08567 upper=5.08567 effort=1.329 velocity=8.26797

Commit message: Cubito supino y actualizado blog

File: pruebas/moving_nao/nao_movement_pattern_creator/Modelo_NAO/nao.urdf (robot description, URDF)
Before this commit: robot NaoH25V50, 79 links, 78 joints
Links:
- link l_ankle: mass 1.16184 -> 2.16184
- link r_ankle: mass 1.16184 -> 2.16184
